File: Pcb/Envirosense/Envirosense.kicad_sch (KiCad schematic)
At the start: 5 parts, among them J1 0.96" OLED, J2 Jack-DC, U2 L7805

Commit message: Pcb
Parts:
- removed U1: ~, ESP32_Footprints:ESP32_30pin, symbol esp32_30pin:ESP32_30Pin
- added U3: ESP32-DEVKIT-V1, ESP32-DEVKIT-V1:MODULE_ESP32_DEVKIT_V1, symbol ESP32-DEVKIT-V1:ESP32-DEVKIT-V1
Connections:
- net +3V3: now also U3.1 (3V3)
- net +5V: now also U3.30 (VIN)
- net GND: now also U3.2 (GND), U3.29 (GND)
- net SCL: now also U3.14 (D22)
- net SDA: now also U3.11 (D21)
